File: headphone-amp/front_panel_circuit_board.kicad_sch (KiCad schematic)
At the start: 10 parts, among them SW501 Mute/unmute, SW502 On/Off toggle

Commit message: Updated headphone-amp kicad project
Parts:
- added C501: C_Polarized, Capacitor_SMD:CP_Elec_6.3x5.8, symbol Device:C_Polarized
- added C502: C, Capacitor_SMD:C_1206_3216Metric_Pad1.33x1.80mm_HandSolder, symbol Device:C
- R501, R502, R503: value 1k -> 2k4
- SW502: value On/Off toggle -> Enable/bypass
Connections:
- net +15V: now also C501.1, C502.1
- net Ground: now also C501.2, C502.2
- net Power_on_cmd renamed Bypass_cmd
Other:
- sheet Toggle circuit for power renamed Toggle circuit for enable-bypass
