File: headphone-amp/headphone-amp.kicad_pcb (KiCad board)
At the start: 2 copper layers, 212 x 145 mm, 85 parts, among them J101 Conn_Coaxial_x2, J102 AudioJack3_Switch, J103 CUI_PD-30, J104 Conn_01x08_Pin, J106 Conn_01x08_Pin, K101 G5V-2, K102 G5V-2, Q201 BD139, Q202 BD140, Q301 BD139, Q302 BD140, Q401 BSS84, Q402 BS170, Q601 BSS84, Q602 BS170, SW501 Mute/unmute, SW502 On/Off toggle, U101 NE5532, U102 NE5532

Commit message: Updated headphone-amp kicad project
Parts:
- removed C106, C107: 2u, Capacitor_THT:C_Axial_L12.0mm_D7.5mm_P15.00mm_Horizontal
- removed K102: G5V-2, Relay_THT:Relay_DPDT_Omron_G5V-2
- removed U102: NE5532, Package_DIP:DIP-8_W7.62mm_LongPads
- added B101: Front-panel, PCM_kikit:Board, F.Cu at (223.1, 21.4)
- added B102: Amplifier, PCM_kikit:Board, F.Cu at (58.6, 17.4)
- added C501: C_Polarized, Capacitor_SMD:CP_Elec_6.3x5.8, F.Cu at (233.3, 118.5)
- added C502: C, Capacitor_SMD:C_1206_3216Metric_Pad1.33x1.80mm_HandSolder, F.Cu at (231.1, 124.2)
- added C701: 10u, Capacitor_THT:C_Axial_L12.0mm_D7.5mm_P15.00mm_Horizontal, F.Cu at (88.0, 86.0)
- added C702: 10u, Capacitor_THT:C_Axial_L12.0mm_D7.5mm_P15.00mm_Horizontal, F.Cu at (88.0, 94.5)
- added C703: 100n, Capacitor_THT:C_Disc_D6.0mm_W2.5mm_P5.00mm, F.Cu at (129.0, 80.5)
- added H101: MountingHole_Pad, MountingHole:MountingHole_4.3mm_M4_DIN965_Pad_TopBottom, F.Cu at (61.5, 25.0)
- added H102: MountingHole_Pad, MountingHole:MountingHole_4.3mm_M4_DIN965_Pad_TopBottom, F.Cu at (185.5, 25.0)
- added H103: MountingHole_Pad, MountingHole:MountingHole_4.3mm_M4_DIN965_Pad_TopBottom, F.Cu at (79.5, 156.0)
- added H104: MountingHole_Pad, MountingHole:MountingHole_4.3mm_M4_DIN965_Pad_TopBottom, F.Cu at (185.5, 155.0)
- added J105: Conn_Coaxial_x2, RCA:rcj-22 vertical RCA, F.Cu at (66.9, 60.5)
- added J107: Conn_01x05_Pin, Connector_Phoenix_GMSTB:PhoenixContact_GMSTB_2,5_5-GF-7,62_1x05_P7.62mm_Horizontal_ThreadedFlange, F.Cu at (61.0, 101.0)
- added JP101: Jumper_2_Small_Open, Connector_PinHeader_2.54mm:PinHeader_2x01_P2.54mm_Vertical, F.Cu at (160.5, 49.8)
- added JP102: Jumper_2_Small_Open, Connector_PinHeader_2.54mm:PinHeader_2x01_P2.54mm_Vertical, F.Cu at (153.0, 49.5)
- added K103: EE2-3NU, Relay_SMD:Relay_DPDT_Kemet_EE2_NU, F.Cu at (80.6, 82.3)
- added R103: 330R, Resistor_THT:R_Axial_DIN0207_L6.3mm_D2.5mm_P10.16mm_Horizontal, F.Cu at (167.4, 77.9)
- added R104: 330R, Resistor_THT:R_Axial_DIN0207_L6.3mm_D2.5mm_P10.16mm_Horizontal, F.Cu at (75.9, 69.0)
- added R701: 1k, Resistor_THT:R_Axial_DIN0207_L6.3mm_D2.5mm_P10.16mm_Horizontal, F.Cu at (106.0, 89.1)
- added R702: 100k, Resistor_THT:R_Axial_DIN0207_L6.3mm_D2.5mm_P10.16mm_Horizontal, F.Cu at (109.5, 78.9)
- added R703: 27k, Resistor_THT:R_Axial_DIN0207_L6.3mm_D2.5mm_P10.16mm_Horizontal, F.Cu at (119.5, 76.4)
- added R704: 10k, Resistor_THT:R_Axial_DIN0207_L6.3mm_D2.5mm_P10.16mm_Horizontal, F.Cu at (116.0, 86.6)
- added R705: 100R, Resistor_THT:R_Axial_DIN0207_L6.3mm_D2.5mm_P10.16mm_Horizontal, F.Cu at (122.4, 76.5)
- added R711: 100k, Resistor_THT:R_Axial_DIN0207_L6.3mm_D2.5mm_P10.16mm_Horizontal, F.Cu at (109.5, 101.6)
- added R712: 1k, Resistor_THT:R_Axial_DIN0207_L6.3mm_D2.5mm_P10.16mm_Horizontal, F.Cu at (106.0, 91.4)
- added R713: 27k, Resistor_THT:R_Axial_DIN0207_L6.3mm_D2.5mm_P10.16mm_Horizontal, F.Cu at (119.5, 102.1)
- added R714: 10k, Resistor_THT:R_Axial_DIN0207_L6.3mm_D2.5mm_P10.16mm_Horizontal, F.Cu at (116.0, 91.9)
- added R715: 100R, Resistor_THT:R_Axial_DIN0207_L6.3mm_D2.5mm_P10.16mm_Horizontal, F.Cu at (133.9, 86.5)
- added U702: OPA2134, Package_DIP:DIP-8_W7.62mm_LongPads, F.Cu at (122.7, 84.2)
- K101: value G5V-2 -> EE2-3NU; footprint Relay_THT:Relay_DPDT_Omron_G5V-2 -> Relay_SMD:Relay_DPDT_Kemet_EE2_NU
- R204, R304: value 6k8 -> 22k
- R501, R502, R503: value 1k -> 2k4
- SW502: value On/Off toggle -> Enable/bypass
- moved D101 64.4 mm to (77.2, 72.5)
- moved D102 57.9 mm to (163.9, 78.7), turned to -90 degrees
- moved K101 51.2 mm to (153.7, 82.4), turned to -90 degrees
- moved J104 4.74 mm to (223.0, 122.5)
- moved R101 3.90 mm to (156.5, 53.6)
- moved H502 2.77 mm to (220.0, 30.2)
- moved H503 1.00 mm to (220.0, 152.0)
Connections:
- net /Front panel circuit board/Power_on_cmd renamed /Front panel circuit board/Bypass_cmd
- net /Front panel circuit board/Toggle circuit for power/SW-bot renamed /Front panel circuit board/Toggle circuit for enable-bypass/SW-bot
- net /Front panel circuit board/Toggle circuit for power/SW-top renamed /Front panel circuit board/Toggle circuit for enable-bypass/SW-top
- J106 pad 7: unconnected-(J106-Pin_7-Pad7) -> Net-(J106-Pin_7)
- J106 pad 8: Net-(D102-K) -> Net-(J106-Pin_8)
- K101 pad 9: unconnected-(K101-Pad9) -> GND
- RV101 pad 3: Net-(C107-Pad2) -> /Preamplifier/Out_R
- RV101 pad 6: Net-(C106-Pad2) -> /Preamplifier/Out_L
Routing:
- net /Front panel circuit board/PE: track 0.00 -> 324.0 mm
- net +15V: track 9.48 -> 253.9 mm
- net Net-(J106-Pin_7): track 0.00 -> 162.4 mm
- net -15V: track 21.6 -> 150.2 mm, vias 0 -> 1
- net Net-(J101-IN2): track 132.7 -> 10.9 mm
- net /Left channel: track 0.00 -> 117.6 mm
- net Net-(J101-IN1): track 112.0 -> 12.8 mm, vias 1 -> 0
- net /Left channel/Out: track 23.6 -> 97.9 mm, vias 2 -> 3
- net Net-(JP102-B): track 16.3 -> 88.4 mm
- net Net-(J106-Pin_8): track 0.00 -> 67.3 mm
- net /Preamplifier/Out_R: track 0.00 -> 59.5 mm
- net /Right channel: track 0.00 -> 57.1 mm
- net /Preamplifier/Out_L: track 0.00 -> 56.3 mm
- net GND: track 35.9 -> 86.2 mm
- net /Right channel/Out: track 22.5 -> 61.0 mm
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- removed copper zone on F.Cu, net GND
Other:
- board size 212 x 145 mm -> 209.5 x 145 mm
