File: headphone-amp/headphone-amp.kicad_sch (KiCad schematic)
At the start: 23 parts, among them J101 Conn_Coaxial_x2, J102 AudioJack3_Switch, J103 CUI_PD-30, J104 Conn_01x08_Pin, J106 Conn_01x08_Pin, J107 Conn_01x05_Pin, K101 G5V-2, K102 G5V-2, U101 NE5532

Commit message: Updated headphone-amp kicad project
Parts:
- removed J103: CUI_PD-30, Connector:CUI_PD-30, symbol Connector:CUI_PD-30
- removed K101, K102: G5V-2, Relay_THT:Relay_DPDT_Omron_G5V-2, symbol Relay:G5V-2
- added B101: Front-panel, PCM_kikit:Board, symbol PCM_kikit:Board
- added B102: Amplifier, PCM_kikit:Board, symbol PCM_kikit:Board
- added J105: Conn_Coaxial_x2, RCA:rcj-22 vertical RCA, symbol Connector:Conn_Coaxial_x2
- added J108: Mini-DIN-4, symbol Connector:Mini-DIN-4
- added JP101, JP102: Jumper_2_Small_Open, Connector_PinHeader_2.54mm:PinHeader_2x01_P2.54mm_Vertical, symbol Jumper:Jumper_2_Small_Open
- added K101, K103: EE2-3NU, Relay_SMD:Relay_DPDT_Kemet_EE2_NU, symbol Relay:EE2-3NU
- added R103, R104: 330R, Resistor_THT:R_Axial_DIN0207_L6.3mm_D2.5mm_P10.16mm_Horizontal, symbol Device:R
- J107: footprint (none) -> Connector_Phoenix_GMSTB:PhoenixContact_GMSTB_2,5_5-GF-7,62_1x05_P7.62mm_Horizontal_ThreadedFlange
Connections:
- net +15V: now also J108.4
- net -15V: now also J108.3
- net GND: now also J105.3 (EXT), J108.1, K101.12, K101.4, K101.9, K103.12
- net Left channel/Out: now also JP102.1 (A)
- net Preamplifier/In_L: now also K103.8
- net Preamplifier/In_R: now also K103.5
- net Preamplifier/Out_L: now also K101.3
- net Preamplifier/Out_R: now also K101.10
- net Right channel/Out: now also JP101.1 (A)
- net at D102.1 (K): now also K101.1, R103.1; no longer J106.8 (Pin_8)
- net at D101.1 (K): now also K103.1, R104.1
- net at J102.R, J102.RN, R102.2: now also JP101.2 (B)
- net at J102.T, J102.TN, R101.2: now also JP102.2 (B)
- net at J101.1 (IN1): now also K103.9
- net at J101.2 (IN2): now also K103.4
- net at J106.7 (Pin_7): now also R104.2
- net Front panel circuit board/Power_on_cmd renamed Front panel circuit board/Bypass_cmd
- new net: J106.8 (Pin_8), R103.2
- new net: J105.1 (IN1), K103.10
- new net: J105.2 (IN2), K103.3
- no-connect marks 4 -> 2
Other:
- sheet Front panel circuit board ports: added Bypass_cmd; removed Power_on_cmd
- note added: "Current limiting resistors for 12V relay coils."
- note added: "High quality signal switching relay. In bypass-mode when not energized."
- moved on the sheet: D102, J101, J102, J107, R101, R102, RV101
