File: headphone-amp/mono-amplifier.kicad_sch (KiCad schematic)
At the start: 19 parts, among them Q301 BD139, Q302 BD140, U101 NE5532

Commit message: Updated headphone-amp kicad project
Parts:
- R304: value 6k8 -> 22k
Changed lines of the file:
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@@
 			)
 		)
-		(property "Value" "6k8"
+		(property "Value" "22k"
 			(at 101.6 96.5199 0)
 			(effects
